Commit message: add core_sim

File: cb_description/urdf/racecar.xacro (robot description, xacro)
@@ -50,5 +50,5 @@
   </link>
   <joint name="$(arg robot_tf_prefix)imu_joint" type="fixed">
-    <origin xyz="0.02 0.0 0.0" rpy="0 0 0"/>
+    <origin xyz="0.0 0.0 0.0" rpy="0 0 0"/>
     <parent link="$(arg robot_tf_prefix)base_link" />
     <child link="$(arg robot_tf_prefix)imu_link" />
